Commit message: Add parent_link param to scout wheel macro for prefix support

File: scout_description/urdf/scout_mini_wheel.xacro (robot description, xacro)
@@ -1,5 +1,5 @@
 <?xml version="1.0"?>
 <robot xmlns:xacro="http://ros.org/wiki/xacro" name="scout_wheel">
-    <xacro:macro name="scout_mini_wheel" params="wheel_prefix *joint_pose">
+    <xacro:macro name="scout_mini_wheel" params="wheel_prefix parent_link:=base_link *joint_pose">
         <link name="${wheel_prefix}_wheel_link">
             <inertial>
@@ -25,5 +25,5 @@
         </link>
         <joint name="${wheel_prefix}_wheel" type="continuous">
-            <parent link="base_link"/>
+            <parent link="${parent_link}"/>
             <child link="${wheel_prefix}_wheel_link"/>
             <xacro:insert_block name="joint_pose"/>
